Commit message: fix the scout_mini car low speed problem and add camera to wpb_home robot, fit the package.xml cannot find in livox_ros_driver2 problem

File: simple_rbt/model/scout/scout_mini.xacro (robot description, xacro)
@@ -36,5 +36,5 @@
                     rpy="1.57 0 -1.57" />
             <geometry>
-                <mesh filename="package://scout_description/meshes/scout_mini_base_link2.dae" />
+                <mesh filename="package://scout_description/meshes/scout_mini_base_link.dae" />
             </geometry>
         </visual>
@@ -111,4 +111,4 @@
     </xacro:scout_mini_wheel_4>
     <xacro:include filename="$(arg urdf_extras)" />
-    <xacro:include filename="$(find scout_description)/urdf/scout_mini.gazebo" />
+    <xacro:include filename="$(find simple_rbt)/model/scout/scout_mini.gazebo" />
 </robot>

Commit message: feat: Integrate Limo and Omni robots into simple_rbt
- Add URDFs, meshes, and Gazebo configs for Limo and Omni robots
- Create modular launch files for each sensor combination (Mid360, Laser+IMU, FrontCam+IMU)
- Add omni_commander.py to parse cmd_vel to Omni 3-wheel motor velocities
- Fix Limo Gazebo control conflicts by removing wheel transmission
- Zero-out Omni initialization offsets and adjust z-height for all sensors
- Update README with usage instructions and upstream project credits

File: simple_rbt/model/scout/scout_mini.xacro (robot description, xacro)
@@ -6,8 +6,8 @@
     <xacro:include filename="$(find simple_rbt)/model/sensor/simple_mid360/model.xacro" />
     <xacro:include filename="$(find simple_rbt)/model/sensor/simple_front_camera/model.xacro" />
-    <xacro:include filename="$(find scout_description)/urdf/scout_mini_wheel_1.xacro" />
-    <xacro:include filename="$(find scout_description)/urdf/scout_mini_wheel_2.xacro" />
-    <xacro:include filename="$(find scout_description)/urdf/scout_mini_wheel_3.xacro" />
-    <xacro:include filename="$(find scout_description)/urdf/scout_mini_wheel_4.xacro" />
+    <xacro:include filename="$(find simple_rbt)/model/scout/urdf/scout_mini_wheel_1.xacro" />
+    <xacro:include filename="$(find simple_rbt)/model/scout/urdf/scout_mini_wheel_2.xacro" />
+    <xacro:include filename="$(find simple_rbt)/model/scout/urdf/scout_mini_wheel_3.xacro" />
+    <xacro:include filename="$(find simple_rbt)/model/scout/urdf/scout_mini_wheel_4.xacro" />
     <xacro:property name="M_PI" value="3.14159"/>
     <xacro:property name="base_x_size" value="0.6200000" />
@@ -36,5 +36,5 @@
                     rpy="1.57 0 -1.57" />
             <geometry>
-                <mesh filename="package://scout_description/meshes/scout_mini_base_link.dae" />
+                <mesh filename="package://simple_rbt/model/scout/meshes/scout_mini_base_link.dae" />
             </geometry>
         </visual>
@@ -68,5 +68,5 @@
                     rpy="0.0 0.0 3.14" />
             <geometry>
-                <mesh filename="package://scout_description/meshes/box_link.STL" />
+                <mesh filename="package://simple_rbt/model/scout/meshes/box_link.STL" />
             </geometry>
             <material name = "red">

File: simple_rbt/model/tracer/tracer_with_front_cam_imu.xacro (robot description, xacro)
@@ -1,5 +1,5 @@
 <?xml version="1.0"?>
 <robot xmlns:xacro="http://www.ros.org/wiki/xacro" name="tracer_with_front_cam_imu">
-  <xacro:include filename="$(find tracer_description)/urdf/tracer_v1.xacro"/>
+  <xacro:include filename="$(find simple_rbt)/model/tracer/urdf/tracer_v1.xacro"/>
   <xacro:include filename="$(find simple_rbt)/model/sensor/simple_front_cam_imu/model.xacro"/>
   <xacro:simple_front_cam_imu

File: simple_rbt/model/tracer/tracer_with_laser_imu.xacro (robot description, xacro)
@@ -1,5 +1,5 @@
 <?xml version="1.0"?>
 <robot xmlns:xacro="http://www.ros.org/wiki/xacro" name="tracer_with_laser_imu">
-  <xacro:include filename="$(find tracer_description)/urdf/tracer_v1.xacro"/>
+  <xacro:include filename="$(find simple_rbt)/model/tracer/urdf/tracer_v1.xacro"/>
   <xacro:include filename="$(find simple_rbt)/model/sensor/simple_laser_imu/model.xacro"/>
   <xacro:simple_laser_imu

File: simple_rbt/model/tracer/tracer_with_mid360.xacro (robot description, xacro)
@@ -1,5 +1,5 @@
 <?xml version="1.0"?>
 <robot xmlns:xacro="http://www.ros.org/wiki/xacro" name="tracer_with_mid360">
-  <xacro:include filename="$(find tracer_description)/urdf/tracer_v1.xacro"/>
+  <xacro:include filename="$(find simple_rbt)/model/tracer/urdf/tracer_v1.xacro"/>
   <xacro:include filename="$(find simple_rbt)/model/sensor/simple_mid360/model.xacro"/>
   <xacro:simple_mid360
