Commit message: feat(simple_rbt): unify sensor namespaces, add battery topic and maze slam launches

File: simple_rbt/model/go2w/go2w.urdf.xacro (robot description, xacro)
@@ -1,4 +1,5 @@
 <?xml version="1.0"?>
 <robot xmlns:xacro="http://ros.org/wiki/xacro" name="go2w">
+  <xacro:arg name="sensor_namespace" default="go2w"/>
   <!-- Gloabal parameters -->
   <xacro:include filename="$(find simple_rbt)/model/go2w/urdf/const.xacro"/>
@@ -299,4 +300,5 @@
     xyz="0.28945 0 -0.046825"
     rpy="${PI} 2.8782 0"
+    sensor_namespace="$(arg sensor_namespace)"
   />
   <!-- Front Camera -->
@@ -305,4 +307,5 @@
     xyz="0.325 0 0.043"
     rpy="0 0 0"
+    sensor_namespace="$(arg sensor_namespace)"
   />
   <xacro:macro name="go2w_transmission" params="joint_name interface">

File: simple_rbt/model/limo/limo_with_front_cam_imu.xacro (robot description, xacro)
@@ -1,6 +1,7 @@
 <?xml version="1.0"?>
 <robot xmlns:xacro="http://www.ros.org/wiki/xacro" name="limo_with_front_cam_imu">
+  <xacro:arg name="sensor_namespace" default="limo"/>
   <xacro:include filename="$(find simple_rbt)/model/limo/urdf/limo_ackerman.xacro"/>
   <xacro:include filename="$(find simple_rbt)/model/sensor/simple_front_cam_imu/model.xacro"/>
-  <xacro:simple_front_cam_imu parent_link="base_link" xyz="0.06 0.0 0.05" rpy="0 0 0" />
+  <xacro:simple_front_cam_imu parent_link="base_link" xyz="0.06 0.0 0.05" rpy="0 0 0" sensor_namespace="$(arg sensor_namespace)" />
 </robot>

File: simple_rbt/model/limo/limo_with_laser_imu.xacro (robot description, xacro)
@@ -1,6 +1,7 @@
 <?xml version="1.0"?>
 <robot xmlns:xacro="http://www.ros.org/wiki/xacro" name="limo_with_laser_imu">
+  <xacro:arg name="sensor_namespace" default="limo"/>
   <xacro:include filename="$(find simple_rbt)/model/limo/urdf/limo_ackerman.xacro"/>
   <xacro:include filename="$(find simple_rbt)/model/sensor/simple_laser_imu/model.xacro"/>
-  <xacro:simple_laser_imu parent_link="base_link" xyz="0.0 0.0 0.05" rpy="0 0 0" />
+  <xacro:simple_laser_imu parent_link="base_link" xyz="0.0 0.0 0.05" rpy="0 0 0" sensor_namespace="$(arg sensor_namespace)" />
 </robot>

File: simple_rbt/model/limo/limo_with_mid360.xacro (robot description, xacro)
@@ -1,4 +1,5 @@
 <?xml version="1.0"?>
 <robot xmlns:xacro="http://www.ros.org/wiki/xacro" name="limo_with_mid360">
+  <xacro:arg name="sensor_namespace" default="limo"/>
   <!-- Include Limo Ackermann Base -->
   <xacro:include filename="$(find simple_rbt)/model/limo/urdf/limo_ackerman.xacro"/>
@@ -9,4 +10,5 @@
     xyz="0.0 0.0 0.05"
     rpy="0 0 0"
+    sensor_namespace="$(arg sensor_namespace)"
   />
 </robot>

File: simple_rbt/model/omni/omni_with_front_cam_imu.xacro (robot description, xacro)
@@ -1,6 +1,7 @@
 <?xml version="1.0"?>
 <robot xmlns:xacro="http://www.ros.org/wiki/xacro" name="omni_with_front_cam_imu">
+  <xacro:arg name="sensor_namespace" default="omni"/>
   <xacro:include filename="$(find simple_rbt)/model/omni/omni_robot.urdf.xacro"/>
   <xacro:include filename="$(find simple_rbt)/model/sensor/simple_front_cam_imu/model.xacro"/>
-  <xacro:simple_front_cam_imu parent_link="base_link" xyz="0.0 0.0 0.05" rpy="0 0 0" />
+  <xacro:simple_front_cam_imu parent_link="base_link" xyz="0.0 0.0 0.05" rpy="0 0 0" sensor_namespace="$(arg sensor_namespace)" />
 </robot>

File: simple_rbt/model/omni/omni_with_laser_imu.xacro (robot description, xacro)
@@ -1,6 +1,7 @@
 <?xml version="1.0"?>
 <robot xmlns:xacro="http://www.ros.org/wiki/xacro" name="omni_with_laser_imu">
+  <xacro:arg name="sensor_namespace" default="omni"/>
   <xacro:include filename="$(find simple_rbt)/model/omni/omni_robot.urdf.xacro"/>
   <xacro:include filename="$(find simple_rbt)/model/sensor/simple_laser_imu/model.xacro"/>
-  <xacro:simple_laser_imu parent_link="base_link" xyz="0.0 0.0 0.05" rpy="0 0 0" />
+  <xacro:simple_laser_imu parent_link="base_link" xyz="0.0 0.0 0.05" rpy="0 0 0" sensor_namespace="$(arg sensor_namespace)" />
 </robot>

File: simple_rbt/model/omni/omni_with_mid360.xacro (robot description, xacro)
@@ -1,4 +1,5 @@
 <?xml version="1.0"?>
 <robot xmlns:xacro="http://www.ros.org/wiki/xacro" name="omni_with_mid360">
+  <xacro:arg name="sensor_namespace" default="omni"/>
   <!-- Include Omni Base -->
   <xacro:include filename="$(find simple_rbt)/model/omni/omni_robot.urdf.xacro"/>
@@ -9,4 +10,5 @@
     xyz="0.0 0.0 0.05"
     rpy="0 0 0"
+    sensor_namespace="$(arg sensor_namespace)"
   />
 </robot>

File: simple_rbt/model/scout/scout_mini.xacro (robot description, xacro)
@@ -3,4 +3,5 @@
     xmlns:xacro="http://ros.org/wiki/xacro">
     <xacro:arg name="robot_namespace" default="/" />
+    <xacro:arg name="sensor_namespace" default="scout" />
     <xacro:arg name="urdf_extras" default="empty.urdf" />
     <xacro:include filename="$(find simple_rbt)/model/sensor/simple_mid360/model.xacro" />
@@ -92,4 +93,5 @@
       xyz="0 0 0.23"
       rpy="0 0 0"
+      sensor_namespace="$(arg sensor_namespace)"
     />
     <xacro:simple_front_camera
@@ -97,4 +99,5 @@
       xyz="0.2 0 0.16"
       rpy="0 0 0"
+      sensor_namespace="$(arg sensor_namespace)"
     />
     <xacro:scout_mini_wheel_1 wheel_prefix="front_left" wheel_diameter="${wheel_diameter}" wheel_width="${wheel_width}">

File: simple_rbt/model/sensor/simple_front_cam_imu/model.xacro (robot description, xacro)
@@ -1,5 +1,5 @@
 <?xml version="1.0"?>
 <robot xmlns:xacro="http://www.ros.org/wiki/xacro">
-    <xacro:macro name="simple_front_cam_imu" params="parent_link xyz rpy">
+    <xacro:macro name="simple_front_cam_imu" params="parent_link xyz rpy sensor_namespace">
         <link name="camera_link">
             <inertial>
@@ -63,7 +63,8 @@
                 </camera>
                 <plugin name="camera_controller" filename="libgazebo_ros_camera.so">
-                    <cameraName>front_camera</cameraName>
-                    <imageTopicName>/camera/image_raw</imageTopicName>
-                    <cameraInfoTopicName>/camera/camera_info</cameraInfoTopicName>
+                    <robotNamespace>${sensor_namespace}</robotNamespace>
+                    <cameraName>camera</cameraName>
+                    <imageTopicName>image_raw</imageTopicName>
+                    <cameraInfoTopicName>camera_info</cameraInfoTopicName>
                     <frameName>camera_link</frameName>
                     <updateRate>30.0</updateRate>
@@ -80,5 +81,6 @@
                 <visualize>true</visualize>
                 <plugin filename="libgazebo_ros_imu_sensor.so" name="imu_plugin">
-                    <topicName>/camera/imu</topicName>
+                    <robotNamespace>${sensor_namespace}</robotNamespace>
+                    <topicName>camera/imu</topicName>
                     <bodyName>imu_link</bodyName>
                     <updateRateHZ>200.0</updateRateHZ>

File: simple_rbt/model/sensor/simple_front_camera/model.xacro (robot description, xacro)
@@ -1,5 +1,5 @@
 <?xml version="1.0"?>
 <robot xmlns:xacro="http://www.ros.org/wiki/xacro">
-    <xacro:macro name="simple_front_camera" params="parent_link xyz rpy">
+    <xacro:macro name="simple_front_camera" params="parent_link xyz rpy sensor_namespace">
         <link name="camera_link">
             <inertial>
@@ -44,7 +44,8 @@
                 </camera>
                 <plugin name="camera_controller" filename="libgazebo_ros_camera.so">
-                    <cameraName>front_camera</cameraName>
-                    <imageTopicName>/camera/image_raw</imageTopicName>
-                    <cameraInfoTopicName>/camera/camera_info</cameraInfoTopicName>
+                    <robotNamespace>${sensor_namespace}</robotNamespace>
+                    <cameraName>camera</cameraName>
+                    <imageTopicName>image_raw</imageTopicName>
+                    <cameraInfoTopicName>camera_info</cameraInfoTopicName>
                     <frameName>camera_link</frameName>
                     <updateRate>30.0</updateRate>

File: simple_rbt/model/sensor/simple_laser_imu/model.xacro (robot description, xacro)
@@ -1,5 +1,5 @@
 <?xml version="1.0"?>
 <robot xmlns:xacro="http://www.ros.org/wiki/xacro">
-    <xacro:macro name="simple_laser_imu" params="parent_link xyz rpy">
+    <xacro:macro name="simple_laser_imu" params="parent_link xyz rpy sensor_namespace">
         <link name="imu_link">
             <inertial>
@@ -64,5 +64,6 @@
                 </ray>
                 <plugin name="gazebo_ros_laser_controller" filename="libgazebo_ros_laser.so">
-                    <topicName>/laser/scan</topicName>
+                    <robotNamespace>${sensor_namespace}</robotNamespace>
+                    <topicName>laser/scan</topicName>
                     <frameName>laser_link</frameName>
                 </plugin>
@@ -76,5 +77,6 @@
                 <visualize>true</visualize>
                 <plugin filename="libgazebo_ros_imu_sensor.so" name="imu_plugin">
-                    <topicName>/laser/imu</topicName>
+                    <robotNamespace>${sensor_namespace}</robotNamespace>
+                    <topicName>laser/imu</topicName>
                     <bodyName>imu_link</bodyName>
                     <updateRateHZ>200.0</updateRateHZ>

File: simple_rbt/model/sensor/simple_mid360/model.xacro (robot description, xacro)
@@ -1,5 +1,5 @@
 <?xml version="1.0"?>
 <robot xmlns:xacro="http://www.ros.org/wiki/xacro">
-    <xacro:macro name="simple_mid360" params="parent_link xyz rpy">
+    <xacro:macro name="simple_mid360" params="parent_link xyz rpy sensor_namespace">
         <link name="livox_link">
             <inertial>
@@ -52,4 +52,5 @@
                 <update_rate>10</update_rate>
                 <plugin name="gazebo_ros_laser_controller" filename="liblivox_laser_simulation.so">
+                    <robotNamespace>${sensor_namespace}</robotNamespace>
                     <ray>
                         <scan>
@@ -83,5 +84,5 @@
                     <csv_file_name>mid360-real-centr.csv</csv_file_name>
                     <publish_pointcloud_type>3</publish_pointcloud_type>
-                    <ros_topic>/livox/lidar</ros_topic>
+                    <ros_topic>livox/lidar</ros_topic>
                     <frameName>livox_link</frameName>
                 </plugin>
@@ -97,5 +98,6 @@
                 <topic>__default_topic__</topic>
                 <plugin filename="libgazebo_ros_imu_sensor.so" name="imu_plugin">
-                    <topicName>/livox/imu</topicName>
+                    <robotNamespace>${sensor_namespace}</robotNamespace>
+                    <topicName>livox/imu</topicName>
                     <bodyName>imu_link</bodyName>
                     <updateRateHZ>200.0</updateRateHZ>

File: simple_rbt/model/tracer/tracer_with_front_cam_imu.xacro (robot description, xacro)
@@ -1,4 +1,5 @@
 <?xml version="1.0"?>
 <robot xmlns:xacro="http://www.ros.org/wiki/xacro" name="tracer_with_front_cam_imu">
+  <xacro:arg name="sensor_namespace" default="tracer"/>
   <xacro:include filename="$(find simple_rbt)/model/tracer/urdf/tracer_v1.xacro"/>
   <xacro:include filename="$(find simple_rbt)/model/sensor/simple_front_cam_imu/model.xacro"/>
@@ -7,4 +8,5 @@
     xyz="0.2 0 0.03"
     rpy="0 0 0"
+    sensor_namespace="$(arg sensor_namespace)"
   />
 </robot>

File: simple_rbt/model/tracer/tracer_with_laser_imu.xacro (robot description, xacro)
@@ -1,4 +1,5 @@
 <?xml version="1.0"?>
 <robot xmlns:xacro="http://www.ros.org/wiki/xacro" name="tracer_with_laser_imu">
+  <xacro:arg name="sensor_namespace" default="tracer"/>
   <xacro:include filename="$(find simple_rbt)/model/tracer/urdf/tracer_v1.xacro"/>
   <xacro:include filename="$(find simple_rbt)/model/sensor/simple_laser_imu/model.xacro"/>
@@ -7,4 +8,5 @@
     xyz="0.0 0 0.03"
     rpy="0 0 0"
+    sensor_namespace="$(arg sensor_namespace)"
   />
 </robot>

File: simple_rbt/model/tracer/tracer_with_mid360.xacro (robot description, xacro)
@@ -1,4 +1,5 @@
 <?xml version="1.0"?>
 <robot xmlns:xacro="http://www.ros.org/wiki/xacro" name="tracer_with_mid360">
+  <xacro:arg name="sensor_namespace" default="tracer"/>
   <xacro:include filename="$(find simple_rbt)/model/tracer/urdf/tracer_v1.xacro"/>
   <xacro:include filename="$(find simple_rbt)/model/sensor/simple_mid360/model.xacro"/>
@@ -7,4 +8,5 @@
     xyz="0.0 0 0.03"
     rpy="0 0 0"
+    sensor_namespace="$(arg sensor_namespace)"
   />
 </robot>
